File: led_clock.sch (KiCad schematic (older format))
At the start: 38 parts, among them M2 LOGO_OSHW, P1 SERIAL, P2 USBCONN, P3 5-9V IN, P4 LEDS, P5 ICSP, P6 CONN_6, Q1 BSS138, Q2 BSS138, Q3 BSS138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

Commit message: Remove references to unused libs/symbols
Parts:
- BT1: symbol BATTERY -> Battery
Changed lines of the file:
@@
 LIBS:contrib
 LIBS:valves
-LIBS:w_opto
 LIBS:RMC
-LIBS:w_microcontrollers
 LIBS:i2sd_v3
 LIBS:opendous
@@
 ROW3
 $Comp
-L BATTERY BT1
+L Battery BT1
 U 1 1 53EFE883
 P 10950 5800
-F 0 "BT1" H 10950 6000 50  0000 C CNN
-F 1 "BATTERY" H 10950 5610 50  0000 C CNN
+F 0 "BT1" H 11100 5950 50  0000 C CNN
+F 1 "BATTERY" H 11150 5700 50  0000 C CNN
 F 2 "w_battery_holders:keystone_106" H 10950 5800 60  0001 C CNN
 F 3 "~" H 10950 5800 60  0000 C CNN
 	1    10950 5800
-	0    1    1    0
+	1    0    0    -1
 $EndComp
 Text Label 8050 6150 0    50   ~ 0
@@
 	9600 6800 9600 6900
 Wire Wire Line
-	9600 6900 10450 6900
+	10450 6900 9600 6900
 Wire Wire Line
 	9700 6800 9700 7000
@@
 	1100 1300 1250 1300
 Wire Wire Line
-	10950 6100 10950 6300
-Wire Wire Line
-	10950 5500 10950 5000
+	10950 5950 10950 6300
+Wire Wire Line
+	10950 5650 10950 5000
 Wire Wire Line
 	10950 5000 9150 5000
